File: PCB/blinktronicator.sch (KiCad schematic (older format))
At the start: 39 parts, among them P1 VCC, P2 GND, P3 RST, P4 SCK, P5 MISO, P6 MOSI, SW2 SW_PUSH, SW3 SW_PUSH, U1 ATTINY85-S, U3 74HC595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

Commit message: many changes. formal name change from "RRRROOOGG..etc" to "blinktronicator". got basic functions working (led update function, mostly). updated PCB to eliminate stupid errors--mirror image shift register footprint, poor programming pad placement, hugely massive round holes for USB plug mounting (they're now slots! and no pads for data lines!), wavelength labels, more?
Parts:
- removed P1: VCC, symbol CONN_1
- removed P2: GND, symbol CONN_1
- D1: value 630nm -> WHT
- D10: value 572nm -> 585nm
- D11: value 566nm -> 590nm
- D12: value 560nm -> 596nm
- D13: value 527nm -> 605nm
- D14: value 470nm -> 615nm
- D15: value pink -> 620nm
- D16: value white -> 630nm
- D2: value 620nm -> PNK
- D3: value 615nm -> 470nm
- D4: value 605nm -> 527nm
- D5: value 596nm -> 560nm
- D6: value 590nm -> 566nm
- D7: value 585nm -> 572nm
- D8: value 580nm -> 576nm
- D9: value 576nm -> 580nm
Connections:
- net labels added: D1, D10, D11, D12, D13, D14, D15, D16, D2, D3, D4, D5, D6, D7, D8, D9
- wire segments 174 -> 142
Other:
- moved on the sheet: D1, D10, D11, D12, D13, D14, D15, D16, D2, D3, D4, D5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
